File: pcb/chiller.sch (KiCad schematic (older format))
At the start: 28 parts, among them IC1 ARDUINO NANO, J1 CONN_01X03, J2 CONN_01X02, J3 CONN_01X02, J4 CONN_01X03, J5 CONN_01X03, J6 CONN_01X03, J7 CONN_01X02, J8 CONN_01X02, J9 CONN_01X02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

Commit message: Finalize schematic.
Parts:
- removed IC1: ARDUINO NANO, symbol arduino:ARDUINO_PRO_MINI_5V
- removed Q1, Q4: MMBT3904, TO_SOT_Packages_SMD:SOT-23, symbol tinkerforge:MMBTA42
- added C4: 100n, Capacitors_SMD:C_0603, symbol chiller-rescue:C
- added C5, C6: 10u, Capacitors_SMD:C_0805, symbol chiller-rescue:C
- added D2: SS34, Diodes_SMD:D_SMC, symbol tinkerforge:D
- added P2: CONN_01X02, Connector_JST:JST_XH_B02B-XH-A_1x02_P2.50mm_Vertical, symbol tinkerforge:CONN_01X02
- added Q1, Q4: BSS138, Package_TO_SOT_SMD:SOT-23, symbol Transistor_FET:BSS138
- added R11, R12, R13, R5, R7, R9: 10K, Resistor_SMD:R_0603_1608Metric, symbol chiller-rescue:R
- added R6, R8: 1K, Resistor_SMD:R_0603_1608Metric, symbol chiller-rescue:R
- added U2: Arduino_Nano_v3.x, Module:Arduino_Nano, symbol MCU_Module:Arduino_Nano_v3.x
- C1: footprint (none) -> Capacitors_SMD:C_0805
- J1: renamed from J4; footprint Connectors_JST:JST_PH_B3B-PH-K_03x2.00mm_Straight -> Connector_JST:JST_XH_B03B-XH-A_1x03_P2.50mm_Vertical
- J10: renamed from J1; footprint Connectors_JST:JST_PH_B3B-PH-K_03x2.00mm_Straight -> Connector_JST:JST_XH_B03B-XH-A_1x03_P2.50mm_Vertical
- J11: renamed from P1; footprint Connectors_JST:JST_PH_B2B-PH-K_02x2.00mm_Straight -> Connector_JST:JST_XH_B02B-XH-A_1x02_P2.50mm_Vertical
- J2: renamed from J5; footprint Connectors_JST:JST_PH_B3B-PH-K_03x2.00mm_Straight -> Connector_JST:JST_XH_B03B-XH-A_1x03_P2.50mm_Vertical
- J3: renamed from J6; footprint Connectors_JST:JST_PH_B3B-PH-K_03x2.00mm_Straight -> Connector_JST:JST_XH_B03B-XH-A_1x03_P2.50mm_Vertical
- J4: renamed from J3; footprint Connectors_JST:JST_PH_B2B-PH-K_02x2.00mm_Straight -> Connector_JST:JST_XH_B02B-XH-A_1x02_P2.50mm_Vertical
- J5: renamed from J9; footprint Connectors_JST:JST_PH_B2B-PH-K_02x2.00mm_Straight -> Connector_JST:JST_XH_B02B-XH-A_1x02_P2.50mm_Vertical
- J6: renamed from J7; footprint Connectors_JST:JST_PH_B2B-PH-K_02x2.00mm_Straight -> Connector_JST:JST_XH_B02B-XH-A_1x02_P2.50mm_Vertical
- J7: renamed from J2; footprint Connectors_JST:JST_PH_B2B-PH-K_02x2.00mm_Straight -> Connector_JST:JST_XH_B02B-XH-A_1x02_P2.50mm_Vertical
- J8: footprint Connectors_JST:JST_PH_B2B-PH-K_02x2.00mm_Straight -> Connector_JST:JST_XH_B02B-XH-A_1x02_P2.50mm_Vertical
- J9: renamed from U2; footprint Pin_Headers:Pin_Header_Straight_1x16_Pitch2.54mm -> Connector_PinHeader_2.54mm:PinHeader_1x16_P2.54mm_Vertical
- R1: footprint Resistors_SMD:R_0603 -> Resistor_SMD:R_0603_1608Metric
- R10: renamed from R2; footprint Resistors_SMD:R_0603 -> Resistor_SMD:R_0603_1608Metric
- R2: renamed from R3; footprint Resistors_SMD:R_0603 -> Resistor_SMD:R_0603_1608Metric
- R3: renamed from R4; footprint Resistors_SMD:R_0603 -> Resistor_SMD:R_0603_1608Metric
- R4: renamed from R5; value R -> 1K; footprint Resistors_SMD:R_0603 -> Resistor_SMD:R_0603_1608Metric
- RL1: value RM50-xx21 -> G6B-1114C-US-DC5; footprint (none) -> libs:DIL-relay
- RV1: footprint (none) -> Potentiometer_SMD:Potentiometer_Vishay_TS53YL_Vertical
Connections:
- net labels added: A0, A1, A2, D10, D11, D12, D2, D9
- wire segments 147 -> 186
- no-connect marks 20 -> 16
Other:
- note added: "CURRENT\nSENSE"
- note added: "POWER"
- moved on the sheet: C3, J10, J4, J5, R4

Commit message: Fix footprints, place all components.
Parts:
- removed RL1: G6B-1114C-US-DC5, libs:DIL-relay, symbol chiller-rescue:RM50-xx21
- added RL1: G6B-1114C-US5DC, modules:DIL-relay, symbol omron:G6B-1114C-US5DC
- U1: footprint libs:DPAK-3 -> modules:DPAK-3
- renumbered P2 to J12
Changed lines of the file:
@@
 F 0 "U1" H 4950 1054 50  0000 C CNN
 F 1 "78M05" H 4800 1450 50  0000 C CNN
-F 2 "libs:DPAK-3" H 4800 1250 50  0001 C CNN
+F 2 "modules:DPAK-3" H 4800 1250 50  0001 C CNN
 F 3 "" H 4800 1250 50  0000 C CNN
 	1    4800 1250
@@
 SSR
 $Comp
-L chiller-rescue:RM50-xx21 RL1
-U 1 1 58D2E664
-P 7800 4400
-F 0 "RL1" H 8250 4550 50  0000 L CNN
-F 1 "G6B-1114C-US-DC5" H 7800 4850 50  0000 L CNN
-F 2 "libs:DIL-relay" H 7800 4400 50  0001 C CNN
-F 3 "" H 7800 4400 50  0001 C CNN
-	1    7800 4400
-	1    0    0    -1
-$EndComp
-$Comp
 L chiller-rescue:POT_TRIM RV1
 U 1 1 58D2E732
@@
 F 3 "" H 9150 4450 50  0001 C CNN
 	1    9150 4450
-	1    0    0    -1
+	1    0    0    1
 $EndComp
 Wire Wire Line
@@
 $EndComp
 $Comp
-L tinkerforge:CONN_01X02 P2
+L tinkerforge:CONN_01X02 J12
 U 1 1 5BC912CA
 P 950 2050
-F 0 "P2" H 869 1775 50  0000 C CNN
+F 0 "J12" H 869 1775 50  0000 C CNN
 F 1 "CONN_01X02" H 869 1866 50  0000 C CNN
 F 2 "Connector_JST:JST_XH_B02B-XH-A_1x02_P2.50mm_Vertical" H 950 1950 50  0001 C CNN
@@
 Wire Wire Line
 	6600 2850 6850 2850
+$Comp
+L omron:G6B-1114C-US5DC RL1
+U 1 1 5BCAFCFB
+P 7800 4400
+F 0 "RL1" H 8230 4446 50  0000 L CNN
+F 1 "G6B-1114C-US5DC" H 8230 4355 50  0000 L CNN
+F 2 "modules:DIL-relay" H 7800 4400 50  0001 C CNN
+F 3 "" H 7800 4400 50  0001 C CNN
+	1    7800 4400
+	1    0    0    -1
+$EndComp
 $EndSCHEMATC

Commit message: Complete routing.
Other:
- note added: "Ready"
- note removed: "LASERSAUR"
Changed lines of the file:
@@
 	8000 4800 8000 4700
 Text Notes 9350 4500 0    60   ~ 0
-LASERSAUR
+Ready
 $Comp
 L chiller-rescue:R R1

Commit message: Make pretty.
Parts:
- C1, C5, C6: footprint Capacitors_SMD:C_0805 -> Capacitor_SMD:C_0805_2012Metric
- C2, C3, C4: footprint Capacitors_SMD:C_0603 -> Capacitor_SMD:C_0603_1608Metric
- D2: footprint Diodes_SMD:D_SMC -> Diode_SMD:D_SMC
Changed lines of the file:
@@
 F 0 "C1" H 4275 1500 50  0000 L CNN
 F 1 "10u" H 4275 1300 50  0000 L CNN
-F 2 "Capacitors_SMD:C_0805" H 4288 1250 50  0001 C CNN
+F 2 "Capacitor_SMD:C_0805_2012Metric" H 4288 1250 50  0001 C CNN
 F 3 "" H 4250 1400 50  0000 C CNN
 	1    4250 1400
@@
 F 0 "C2" H 5275 1500 50  0000 L CNN
 F 1 "100n" H 5275 1300 50  0000 L CNN
-F 2 "Capacitors_SMD:C_0603" H 5288 1250 50  0001 C CNN
+F 2 "Capacitor_SMD:C_0603_1608Metric" H 5288 1250 50  0001 C CNN
 F 3 "" H 5250 1400 50  0000 C CNN
 	1    5250 1400
@@
 F 0 "C3" H 5675 2050 50  0000 L CNN
 F 1 "100n" H 5675 1850 50  0000 L CNN
-F 2 "Capacitors_SMD:C_0603" H 5688 1800 50  0001 C CNN
+F 2 "Capacitor_SMD:C_0603_1608Metric" H 5688 1800 50  0001 C CNN
 F 3 "" H 5650 1950 50  0001 C CNN
 	1    5650 1950
@@
 F 0 "C5" H 7100 4500 50  0000 L CNN
 F 1 "10u" H 7250 4500 50  0000 L CNN
-F 2 "Capacitors_SMD:C_0805" H 7238 4150 50  0001 C CNN
+F 2 "Capacitor_SMD:C_0805_2012Metric" H 7238 4150 50  0001 C CNN
 F 3 "" H 7200 4300 50  0001 C CNN
 	1    7200 4300
@@
 F 0 "C4" V 7098 1350 50  0000 C CNN
 F 1 "100n" V 7189 1350 50  0000 C CNN
-F 2 "Capacitors_SMD:C_0603" H 7388 1200 50  0001 C CNN
+F 2 "Capacitor_SMD:C_0603_1608Metric" H 7388 1200 50  0001 C CNN
 F 3 "" H 7350 1350 50  0001 C CNN
 	1    7350 1350
@@
 F 0 "D2" V 3804 6478 50  0000 L CNN
 F 1 "SS34" V 3895 6478 50  0000 L CNN
-F 2 "Diodes_SMD:D_SMC" H 3850 6400 50  0001 C CNN
+F 2 "Diode_SMD:D_SMC" H 3850 6400 50  0001 C CNN
 F 3 "" H 3850 6400 50  0000 C CNN
 	1    3850 6400
@@
 F 0 "C6" H 1415 2796 50  0000 L CNN
 F 1 "10u" H 1415 2705 50  0000 L CNN
-F 2 "Capacitors_SMD:C_0805" H 1338 2600 50  0001 C CNN
+F 2 "Capacitor_SMD:C_0805_2012Metric" H 1338 2600 50  0001 C CNN
 F 3 "" H 1300 2750 50  0001 C CNN
 	1    1300 2750
