File: pcb/chiller.kicad_sch (KiCad schematic)
At the start: 58 parts, among them J1 Temp sensor 1, J10 Current Sense, J11 Display, J12 Debug, J13 Conn_01x04, J14 Flow sensor, J15 Fan, J16 Buzzer, J2 Temp sensor 2, J3 Ext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

Commit message: Route.
Parts:
- removed J10: Current Sense, Connector_JST:JST_XH_B3B-XH-A_1x03_P2.50mm_Vertical, symbol Connector_Generic:Conn_01x03
- J16: footprint (none) -> Connector_JST:JST_XH_B2B-XH-A_1x02_P2.50mm_Vertical
- J3: footprint Connector_PinHeader_2.54mm:PinHeader_1x04_P2.54mm_Vertical -> Connector_PinHeader_2.54mm:PinHeader_1x05_P2.54mm_Vertical; symbol Connector_Generic:Conn_01x04 -> Connector_Generic:Conn_01x05
- Q6: footprint Package_TO_SOT_SMD:SOT-23 -> Package_TO_SOT_SMD:SOT-223-3_TabPin2
- R8: value 2k2 -> 33k
- R9: value 1k2 -> 18k
- SW1, SW2: footprint (none) -> Button_Switch_SMD:SW_SPST_CK_RS282G05A3
- renumbered J15 to J10
Connections:
- net Ext1: now also J3.4 (Pin_4); no longer J3.3 (Pin_3)
- net Ext2: now also J3.3 (Pin_3); no longer J3.2 (Pin_2)
- net GND: now also J3.5 (Pin_5); no longer J3.4 (Pin_4)
- net CurrentSense renamed Ext3
- net Ext3: now also J3.2 (Pin_2)
