File: pcb/addon/addon.kicad_pcb (KiCad board)
At the start: 2 copper layers, 38.1 x 43.2 mm, 12 parts, among them J1 12V in, J2 Fan out, J3 Fan control, J4 Ext, J5 Buzzer, Q1 BC547, Q2 IRFZ44N

Commit message: Add more test commands.
Parts:
- R1: footprint Resistor_THT:R_Axial_DIN0207_L6.3mm_D2.5mm_P10.16mm_Horizontal -> Resistor_THT:R_Axial_DIN0204_L3.6mm_D1.6mm_P7.62mm_Horizontal
- R3: footprint Resistor_THT:R_Axial_DIN0207_L6.3mm_D2.5mm_P10.16mm_Horizontal -> Resistor_THT:R_Axial_DIN0207_L6.3mm_D2.5mm_P7.62mm_Horizontal
- moved R3 2.54 mm to (121.9, 99.1)
Routing:
- net GND: track 83.9 -> 81.3 mm
- net Net-(J4-Pin_3): track 5.11 -> 7.65 mm
- net Net-(Q2-G): track 17.8 -> 20.3 mm

Commit message: Finalize.
Other:
- board text added: "12V IN"
- board text added: "BUZZER"
- board text added: "FAN CONTROL"
- board text added: "FAN OUT"
Changed lines of the file:
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@@
     (descr "Resistor, Axial_DIN0204 series, Axial, Horizontal, pin pitch=7.62mm, 0.167W, length*diameter=3.6*1.6mm^2, http://cdn-reichelt.de/documents/datenblatt/B400/1_4W%23YAG.pdf")
     (tags "Resistor Axial_DIN0204 series Axial Horizontal pin pitch 7.62mm 0.167W length 3.6mm diameter 1.6mm")
-    (property "Reference" "R1" (at 3.81 -1.92 0) (layer "F.SilkS")
-      (effects (font (size 1 1) (thickness 0.15)))
-    )
-    (property "Value" "1k" (at 3.81 1.92 0) (layer "F.Fab")
+    (property "Reference" "R1" (at 3.81 -1.92 0) (layer "F.SilkS") hide
+      (effects (font (size 1 1) (thickness 0.15)))
+    )
+    (property "Value" "1k" (at 3.81 1.92 0) (layer "F.Fab") hide
       (effects (font (size 1 1) (thickness 0.15)))
     )
@@
     (descr "Resistor, Axial_DIN0207 series, Axial, Horizontal, pin pitch=7.62mm, 0.25W = 1/4W, length*diameter=6.3*2.5mm^2, http://cdn-reichelt.de/documents/datenblatt/B400/1_4W%23YAG.pdf")
     (tags "Resistor Axial_DIN0207 series Axial Horizontal pin pitch 7.62mm 0.25W = 1/4W length 6.3mm diameter 2.5mm")
-    (property "Reference" "R3" (at 3.81 -2.37 0) (layer "F.SilkS")
-      (effects (font (size 1 1) (thickness 0.15)))
-    )
-    (property "Value" "2k2" (at 3.81 2.37 0) (layer "F.Fab")
+    (property "Reference" "R3" (at 3.81 -2.37 0) (layer "F.SilkS") hide
+      (effects (font (size 1 1) (thickness 0.15)))
+    )
+    (property "Value" "2k2" (at 3.81 2.37 0) (layer "F.Fab") hide
       (effects (font (size 1 1) (thickness 0.15)))
     )
@@
   (gr_rect (start 109.22 63.5) (end 147.32 106.68)
     (stroke (width 0.1) (type default)) (fill none) (layer "Edge.Cuts"))
+  (gr_text "FAN\nCONTROL" (at 101.6 86.106 0) (layer "F.SilkS")
+    (effects (font (size 1 1) (thickness 0.15)) (justify left bottom))
+  )
+  (gr_text "BUZZER" (at 148.59 80.772 0) (layer "F.SilkS")
+    (effects (font (size 1 1) (thickness 0.15)) (justify left bottom))
+  )
+  (gr_text "12V IN" (at 101.854 70.358 0) (layer "F.SilkS")
+    (effects (font (size 1 1) (thickness 0.15)) (justify left bottom))
+  )
+  (gr_text "FAN OUT" (at 148.082 70.104 0) (layer "F.SilkS")
+    (effects (font (size 1 1) (thickness 0.15)) (justify left bottom))
+  )
   (segment (start 132.08 66.04) (end 137.16 66.04) (width 1) (layer "F.Cu") (net 1))
   (segment (start 132.08 73.66) (end 127 73.66) (width 1) (layer "F.Cu") (net 1))
